File: panel/OpenRX-panel-rev2.2.kicad_pcb (KiCad board)
At the start: 6 copper layers, 64.2 x 17.3 mm, 242 parts, among them J1 Conn_Coaxial_Small, J101 Conn_Coaxial_Small, J2 Conn_Coaxial_Small, J201 Conn_Coaxial, T1 0900PC16J0042001E, T101 0900PC16J0042001E, T2 0900PC16J0042001E, U1 ESP32-C3, U101 ESP32-C3, U102 TLV75533PDQNR, U103 LR1121IMLTRT, U104 RFX2401C, U105 SKY13373-460LF, U2 TLV75533PDQNR, U201 ESP32-C3, U202 TLV75533PDQNR, U203 SX1281IMLTRT, U3 LR1121IMLTRT, U301 ESP32-C3, U302 TLV75533PDQNR, U303 SX1281IMLTRT, U4 RFX2401C, U5 SKY13373-460LF, U6 LR1121IMLTRT, U7 RFX2401C, U8 SKY13373-460LF, U9 TS2306A 240GF MSM 9_C2976675, X1 CJ17-400001010B20, X101 CJ17-400001010B20, X201 CJ17-400001010B20, X301 CJ17-400001010B20

Commit message: Panel carries its own breakaway webs and mouse bites (#55)
4-in-1 panel with its own breakaway webs and mouse bites (frame from 0459acc), copper keepouts on the webs.

Co-Authored-By: Claude Opus 5.5 <noreply@anthropic.com>
Parts:
- added REF**: BreakLine_5h_D0.5mm_P0.85mm, Panelization:BreakLine_5h_D0.5mm_P0.85mm, F.Cu at (153.9, 109.5)
- added REF**: BreakLine_11h_D0.5mm_P0.85mm, Panelization:BreakLine_11h_D0.5mm_P0.85mm, F.Cu at (117.2, 106.8)
- added REF**: BreakLine_5h_D0.5mm_P0.85mm, Panelization:BreakLine_5h_D0.5mm_P0.85mm, F.Cu at (148.4, 109.5)
- added REF**: BreakLine_5h_D0.5mm_P0.85mm, Panelization:BreakLine_5h_D0.5mm_P0.85mm, F.Cu at (137.9, 114.0)
- added REF**: BreakLine_5h_D0.5mm_P0.85mm, Panelization:BreakLine_5h_D0.5mm_P0.85mm, F.Cu at (132.9, 109.5)
- added REF**: BreakLine_5h_D0.5mm_P0.85mm, Panelization:BreakLine_5h_D0.5mm_P0.85mm, F.Cu at (148.4, 114.0)
- added REF**: BreakLine_5h_D0.5mm_P0.85mm, Panelization:BreakLine_5h_D0.5mm_P0.85mm, F.Cu at (122.4, 114.0)
- added REF**: BreakLine_5h_D0.5mm_P0.85mm, Panelization:BreakLine_5h_D0.5mm_P0.85mm, F.Cu at (117.2, 114.0)
- added REF**: BreakLine_5h_D0.5mm_P0.85mm, Panelization:BreakLine_5h_D0.5mm_P0.85mm, F.Cu at (153.9, 114.0)
- added REF**: BreakLine_5h_D0.5mm_P0.85mm, Panelization:BreakLine_5h_D0.5mm_P0.85mm, F.Cu at (132.9, 114.0)
- added REF**: BreakLine_11h_D0.5mm_P0.85mm, Panelization:BreakLine_11h_D0.5mm_P0.85mm, F.Cu at (122.4, 106.8)
- added REF**: BreakLine_5h_D0.5mm_P0.85mm, Panelization:BreakLine_5h_D0.5mm_P0.85mm, F.Cu at (137.9, 109.5)
Other:
- outline, holes or cut-outs redrawn
